Commit message: feat: update pincher mesh and collision parameters; add CAD lenses to simulation

File: src/z70_description/urdf/pincher_collisions.xacro (robot description, xacro)
@@ -2,7 +2,7 @@
   <xacro:macro name="arm_wrist_link_collisions">
     <collision>
-      <origin xyz="0.0138 0 -0.00175732744058" />
+      <origin xyz="0.0138 0 -0.00185" />
       <geometry>
-        <box size="0.067 0.032 0.0215146548812" />
+        <box size="0.067 0.032 0.0217" />
       </geometry>
     </collision>
